File: electronics_brushknight_esp32s3/panel/base/1x1.kicad_pcb (KiCad board)
At the start: 4 copper layers, 96 x 96 mm, 267 parts, among them J1 BLDC, J2 USB_C_Receptacle_USB2.0, J3 LCD, J4 A, J5 B, J6 LCD - FPC, J7 Conn_01x04_Socket, J8 Conn_01x04_Socket, J9 Conn_01x04_Socket, Q1 MMBT4403, Q2 BSS138, Q3 BSS138, SW1 RST, SW2 Boot, U1 MT6701-CT, U10 ESP32-S3-WROOM-1-N8R8, U2 USBLC6-2SC6, U3 VL53L0CXV0DH_1, U4 HX711, U5 TMC6300, U6 LP5907MFX-2.8, U7 SN74LV1T34DBV, U8 VEML7700, U9 TS1117BCW33_RPG

Commit message: minor changes for PCBs order
Parts:
- removed the C11 at (68.8, 108.2)
- removed the C11 at (110.1, 72.8)
- removed Z5: dummy_keepouts, view_custom:ViewKeepouts3d
- added C11: 0.1uF, cleaned footprints:C_0603_1608Metric, F.Cu at (68.8, 108.2)
- added C11: 0.1uF, cleaned footprints:C_0402_1005Metric, F.Cu at (110.1, 72.8)
- added REF**: Fiducial_1mm_Mask3mm, Fiducial:Fiducial_1mm_Mask3mm, B.Cu at (108.0, 29.5)
- added REF**: Fiducial_1mm_Mask3mm, Fiducial:Fiducial_1mm_Mask3mm, B.Cu at (62.0, 29.5)
- added REF**: Fiducial_1mm_Mask3mm, Fiducial:Fiducial_1mm_Mask3mm, B.Cu at (39.5, 52.0)
- added REF**: Fiducial_1mm_Mask3mm, Fiducial:Fiducial_1mm_Mask3mm, B.Cu at (39.5, 98.0)
- added REF**: seedlabs_smartknob, seedlabs:seedlabs_smartknob, F.Cu at (113.5, 43.0)
- added TP17: IO40, cleaned footprints:TestPoint_Pad_D2.0mm_ValueSilk, B.Cu at (101.2, 113.2)
- added TP18: IO41, cleaned footprints:TestPoint_Pad_D2.0mm_ValueSilk, B.Cu at (98.2, 113.2)
- added TP19: IO42, cleaned footprints:TestPoint_Pad_D2.0mm_ValueSilk, B.Cu at (95.2, 113.2)
- added TP20: IO45, cleaned footprints:TestPoint_Pad_D2.0mm_ValueSilk, B.Cu at (104.2, 113.2)
- added TP21: IO46, cleaned footprints:TestPoint_Pad_D2.0mm_ValueSilk, B.Cu at (113.2, 113.2)
- added TP22: IO47, cleaned footprints:TestPoint_Pad_D2.0mm_ValueSilk, B.Cu at (110.2, 113.2)
- added TP23: IO48, cleaned footprints:TestPoint_Pad_D2.0mm_ValueSilk, B.Cu at (107.2, 113.2)
- added Z10: BLDCMotor, BOM_Only:bom_only_no_pin, F.Cu at (121.9, 71.8)
- added Z6: RotorScrew (BOM-only), BOM_Only:bom_only_no_pin, F.Cu at (120.4, 71.8)
- added Z7: RotorScrew (BOM-only), BOM_Only:bom_only_no_pin, F.Cu at (121.9, 71.8)
- added Z8: RotorScrew (BOM-only), BOM_Only:bom_only_no_pin, F.Cu at (123.4, 71.8)
- added Z9: WatchGlass39.5mm, BOM_Only:bom_only_no_pin, F.Cu at (120.4, 71.8)
- moved TP1 2.71 mm to (116.2, 113.2)
- moved TP3 1.71 mm to (119.2, 113.2)
- moved TP2 0.71 mm to (122.2, 113.2)
Connections:
- U10 pad 16: unconnected-(U10-IO46-Pad16) -> Net-(U10-IO46)
- U10 pad 24: unconnected-(U10-IO47-Pad24) -> Net-(U10-IO47)
- U10 pad 25: unconnected-(U10-IO48-Pad25) -> Net-(U10-IO48)
- U10 pad 26: unconnected-(U10-IO45-Pad26) -> Net-(U10-IO45)
- U10 pad 33: unconnected-(U10-IO40-Pad33) -> Net-(U10-IO40)
- U10 pad 34: unconnected-(U10-IO41-Pad34) -> Net-(U10-IO41)
- U10 pad 35: unconnected-(U10-IO42-Pad35) -> Net-(U10-IO42)
Routing:
- net Net-(U10-IO46): track 0.00 -> 104.6 mm, vias 0 -> 2
- net Net-(U10-IO47): track 0.00 -> 93.0 mm, vias 0 -> 2
- net Net-(U10-IO48): track 0.00 -> 91.2 mm, vias 0 -> 2
- net Net-(U10-IO45): track 0.00 -> 87.4 mm, vias 0 -> 2
- net Net-(U10-IO40): track 0.00 -> 76.1 mm, vias 0 -> 2
- net Net-(U10-IO41): track 0.00 -> 72.2 mm, vias 0 -> 2
- net Net-(U10-IO42): track 0.00 -> 68.0 mm, vias 0 -> 2
- net +5V: track 69.6 -> 79.1 mm, vias 77 -> 78
- net /ESP32_BOOT: track 48.1 -> 56.1 mm, vias 2 -> 5
- net GNDA: track 79.5 -> 84.1 mm
- net /LED_DATA_3V3: track 34.7 -> 38.7 mm
- net /LCD_CMD: track 29.7 -> 32.7 mm
- net /ESP32_EN: track 18.8 -> 16.0 mm
- net /USB_SERIAL_TXO: track 16.0 -> 18.7 mm
- net /USB_SERIAL_RXI: track 11.5 -> 14.0 mm
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Other:
- outline, holes or cut-outs redrawn
- board text added: "DEVKIT"
- board text added: "JLCJLCJLCJLC"
- board text added: "V-CUT"
- board text added: "v0.1"
- board text removed: "SmartKnob DevKit"
- board text removed: "esp32s3"
