File: electronics_brushknight_esp32s3/view_screen/view_screen.kicad_pcb (KiCad board)
At the start: 4 copper layers, 35 x 35 mm, 14 parts, among them J1 Conn_01x04, J2 GC9A01, J3 Conn_01x04, J4 Conn_01x04, J5 Conn_01x04, J6 LCD - FPC, Q1 2N7002

Commit message: silkscreen fixes
Other:
- board text added: "Screen PCB"
- board text removed: "Screen PCB ${RELEASE_VERSION}"
Changed lines of the file:
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@@
         (effects (font (size 1 1) (thickness 0.15)) (justify mirror))
     )
-    (fp_text value "GC9A01" (at 0 0.5 90) (layer "B.Fab")
+    (fp_text value "GC9A01" (at 0 0.5 90) (layer "B.Fab") hide
         (effects (font (size 1 1) (thickness 0.15)) (justify mirror))
     )
@@
     (property "ki_keywords" "connector")
     (attr smd)
-    (fp_text reference "J6" (at 7.975 0.85 135 unlocked) (layer "B.SilkS")
+    (fp_text reference "J6" (at 7.975 0.85 135 unlocked) (layer "B.SilkS") hide
         (effects (font (size 1 1) (thickness 0.1)) (justify mirror))
     )
-    (fp_text value "LCD - FPC" (at 7.975 -0.65 135 unlocked) (layer "B.Fab")
-        (effects (font (size 1 1) (thickness 0.15)) (justify mirror))
-    )
-    (fp_text user "${REFERENCE}" (at 7.975 -2.15 135 unlocked) (layer "B.Fab")
+    (fp_text value "LCD - FPC" (at 7.975 -0.65 135 unlocked) (layer "B.Fab") hide
+        (effects (font (size 1 1) (thickness 0.15)) (justify mirror))
+    )
+    (fp_text user "${REFERENCE}" (at 7.975 -2.15 135 unlocked) (layer "B.Fab") hide
         (effects (font (size 1 1) (thickness 0.15)) (justify mirror))
     )
@@
     (effects (font (size 1 1) (thickness 0.15)) (justify mirror))
   )
-  (gr_text "Screen PCB\n${RELEASE_VERSION}" (at 117 99.6) (layer "B.SilkS")
+  (gr_text "Screen PCB\n" (at 117 98.75) (layer "B.SilkS")
     (effects (font (size 1 1) (thickness 0.1)) (justify left mirror))
   )
