File: electronics_brushknight_esp32s3/view_screen/view_screen.kicad_pcb (KiCad board)
At the start: 2 copper layers, 35 x 35 mm, 12 parts, among them J1 Conn_01x04, J2 GC9A01, J3 Conn_01x04, J4 Conn_01x04, J5 Conn_01x04, Q1 2N7002

Commit message: devkit pcb preview
Parts:
- added J6: LCD - FPC, screen_connector:Amphenol FCI FPC 8 pin 0.5 pitch, B.Cu at (90.2, 109.8)
- added REF**: fpc_wire_hole_6mm, view_custom:fpc_wire_hole_6mm, F.Cu at (93.0, 107.0)
Routing:
- net /BACKLIGHT_EN: track 21.2 -> 54.5 mm, vias 1 -> 3
- net /DC: track 30.7 -> 49.0 mm, vias 1 -> 3
- net /SCK: track 26.4 -> 39.3 mm, vias 1 -> 4
- net /nCS: track 21.9 -> 34.4 mm, vias 1 -> 4
- net /MOSI: track 31.0 -> 39.9 mm, vias 1 -> 4
- net GND: track 0.00 -> 7.92 mm, vias 13 -> 12
- net /nRESET: track 35.5 -> 41.2 mm, vias 1 -> 3
- net /VDD: track 27.2 -> 30.7 mm, vias 1 -> 3
- added copper zone on In1.Cu, net /VDD
- added copper zone on In2.Cu, net GND
- removed copper zone on B.Cu, net GND
- removed copper zone on F.Cu, net GND
Other:
- copper layers 2 -> 4
- board text added: "Screen PCB"
- board text removed: "COMMIT: ${COMMIT_HASH} DATE: ${COMMIT_DATE}"
- board text removed: "Screen PCB ${RELEASE_VERSION}"
